File: npn-pnp-h-bridge.kicad_sch (KiCad schematic)
At the start: 53 parts, among them J1 S4B-PH-K-S_LF__SN_, J2 S2B-PH-K-S_LF__SN_

Commit message: dont know what im doing
Parts:
- removed C1, C2: 100p, Capacitor_SMD:C_0805_2012Metric_Pad1.18x1.45mm_HandSolder, symbol PCM_Elektuur:C
- removed Qh2: BD140, Package_TO_SOT_THT:TO-126-3_Vertical, symbol Transistor_BJT:BD140
- removed Ql2: BD139, Package_TO_SOT_THT:TO-126-3_Vertical, symbol Transistor_BJT:BD139
- removed Ql3, Ql4: MMBT3904, Package_TO_SOT_SMD:SOT-23, symbol Transistor_BJT:MMBT3904
- removed R13, R9: 3.3k, Resistor_SMD:R_0805_2012Metric_Pad1.20x1.40mm_HandSolder, symbol PCM_Elektuur:R
- added Qh2: BC327, Package_TO_SOT_THT:TO-92_Inline, symbol Transistor_BJT:BC327
- added Ql2: BC337, Package_TO_SOT_THT:TO-92_Inline, symbol Transistor_BJT:BC337
- Qh1: value BD140 -> BC327; footprint Package_TO_SOT_THT:TO-126-3_Vertical -> Package_TO_SOT_THT:TO-92_Inline; symbol Transistor_BJT:BD140 -> Transistor_BJT:BC327
- Ql1: value BD139 -> BC337; footprint Package_TO_SOT_THT:TO-126-3_Vertical -> Package_TO_SOT_THT:TO-92_Inline; symbol Transistor_BJT:BD139 -> Transistor_BJT:BC337
- R10, R14: value 2.2k -> 10k
Connections:
- net +5V: now also Qh1.3 (E), Qh2.3 (E); no longer Qh1.1 (E)
- net GND: now also Ql1.3 (E), Ql2.3 (E); no longer Ql1.1 (E)
- net H1b: now also Qh1.2 (B), R10.1 (+); no longer Qh1.3 (B)
- net H2b: now also R14.1 (+), Qh2.2 (B)
- net HI : now also J1.3, V4.1; no longer R10.1 (+)
- net L1b: now also Ql1.2 (B); no longer Ql1.3 (B)
- net L2b: now also Ql2.2 (B)
- net LO: now also J1.4, V5.1; no longer R14.1 (+)
- net O1: now also Qh1.1 (C), Ql1.1 (C); no longer Qh1.2 (C), Ql1.2 (C)
- net O2: now also Qh2.1 (C), Ql2.1 (C)
- net HI_IN: no longer names the net of V1.1
- net HI_IN: no longer J1.3
- net LO_IN: no longer names the net of V2.1
- net LO_IN: no longer J1.4
Other:
- moved on the sheet: R1, R10, R14

Commit message: sort of working
Parts:
- removed R10, R14: 10k, Resistor_SMD:R_0805_2012Metric_Pad1.20x1.40mm_HandSolder, symbol PCM_Elektuur:R
- added Q1, Q3: AO3400A, Package_TO_SOT_SMD:SOT-23, symbol Transistor_FET:AO3400A
- added R4, R6: 1k, Resistor_SMD:R_0805_2012Metric_Pad1.20x1.40mm_HandSolder, symbol PCM_Elektuur:R
- added R5, R8: 100, Resistor_SMD:R_0805_2012Metric_Pad1.20x1.40mm_HandSolder, symbol PCM_Elektuur:R
- added R9: 10, Resistor_SMD:R_0805_2012Metric_Pad1.20x1.40mm_HandSolder, symbol PCM_Elektuur:R
- added V8: 3.3, symbol Simulation_SPICE:VDC
- R1, R7: value 2.2k -> 1k
Connections:
- net +5V: now also R5.1 (+), R8.1 (+)
- net GND: now also V8.2
- net H1b: now also R1.1 (+), R2.1 (+), Q3.3 (D), R5.2 (-); no longer Qh1.2 (B), R1.2 (-)
- net LO: now also Q1.3 (D), R8.2 (-); no longer J1.4, V5.1
- net O1: now also R9.1 (+); no longer D1.2 (A), D10.2 (A), D11.2 (A), D12.1 (K), D13.2 (A), D14.1 (K), D15.2 (A), D16.1 (K), D17.2 (A), D18.1 (K), D19.2 (A), D2.1 (K), D20.1 (K), D21.2 (A), D22.1 (K), D23.2 (A), D24.2 (A), D25.1 (K), D26.2 (A), D27.1 (K), D28.2 (A), D29.1 (K), D3.2 (A), D30.2 (A), D4.1 (K), D5.1 (K), D6.2 (A), D7.1 (K), D8.2 (A), D9.1 (K)
- net HI_IN: now reaches V1.1
- net HI_IN: now also J1.3, Q3.2 (S), R4.2 (-)
- net LO_IN: now reaches V2.1
- net LO_IN: now also J1.4, Q1.2 (S), R6.2 (-)
- removed net HI : J1.3, R1.1 (+), R2.1 (+), V4.1
- new net: D1.2 (A), D10.2 (A), D11.2 (A), D12.1 (K), D13.2 (A), D14.1 (K), D15.2 (A), D16.1 (K), D17.2 (A), D18.1 (K), D19.2 (A), D2.1 (K), D20.1 (K), D21.2 (A), D22.1 (K), D23.2 (A), D24.2 (A), D25.1 (K), D26.2 (A), D27.1 (K), D28.2 (A), D29.1 (K), D3.2 (A), D30.2 (A), D4.1 (K), D5.1 (K), D6.2 (A), D7.1 (K), D8.2 (A), D9.1 (K), R9.2 (-)
- new net: Qh1.2 (B), R1.2 (-)
- new net +3.3V: Q1.1 (G), Q3.1 (G), R4.1 (+), R6.1 (+), V8.1
Other:
- moved on the sheet: J2, Qh1, Qh2, Ql1, Ql2, R1, R2, R3, R7

Commit message: sorta working
Parts:
- removed D24, D3: LED, LED_THT:LED_D5.0mm, symbol Device:LED
- removed R9: 10, Resistor_SMD:R_0805_2012Metric_Pad1.20x1.40mm_HandSolder, symbol PCM_Elektuur:R
- added C1, C2: 100p, Capacitor_SMD:C_0805_2012Metric_Pad1.18x1.45mm_HandSolder, symbol PCM_Elektuur:C
- added Q2, Q4: MMBT3904, Package_TO_SOT_SMD:SOT-23, symbol Transistor_BJT:MMBT3904
- added R10, R13: 1k, Resistor_SMD:R_0805_2012Metric_Pad1.20x1.40mm_HandSolder, symbol PCM_Elektuur:R
- added R11, R12, R16, R17: 10k, Resistor_SMD:R_0805_2012Metric_Pad1.20x1.40mm_HandSolder, symbol PCM_Elektuur:R
- added R14, R15: 100, Resistor_SMD:R_0805_2012Metric_Pad1.20x1.40mm_HandSolder, symbol PCM_Elektuur:R
- added R19, R20, R21, R22, R23, R25, R26, R27, R28, R29, R30, R31, R33, R34, R35, R36, R37, R38, R39, R40, R41, R42, R43, R44, R45, R46, R47, R48: 330, Resistor_SMD:R_0805_2012Metric_Pad1.20x1.40mm_HandSolder, symbol PCM_Elektuur:R
Connections:
- net +5V: now also R11.2 (-), R12.2 (-), R14.2 (-), R15.2 (-)
- net GND: now also Q2.2 (E), Q4.2 (E), R16.1 (+), R17.1 (+)
- net H1b: now also Q2.3 (C), R15.1 (+)
- net H2b: now also R12.1 (+)
- net HI_IN: now also C1.1 (+), R10.1 (+)
- net L1b: now also R16.2 (-)
- net L2b: now also R17.2 (-)
- net LO: now also Q4.3 (C), R14.1 (+)
- net LO_IN: now also C2.1 (+), R13.1 (+)
- net O1: now also D12.1 (K), D14.1 (K), D16.1 (K), D18.1 (K), D2.1 (K), D20.1 (K), D22.1 (K), D25.1 (K), D27.1 (K), D29.1 (K), D4.1 (K), D5.1 (K), D7.1 (K), D9.1 (K), R20.1 (+), R21.1 (+), R22.1 (+), R23.1 (+), R25.1 (+), R26.1 (+), R27.1 (+), R28.1 (+), R29.1 (+), R30.1 (+), R31.1 (+), R33.1 (+), R34.1 (+), R35.1 (+)
- net O2: now also R19.2 (-), R36.2 (-), R37.2 (-), R38.2 (-), R39.2 (-), R40.2 (-), R41.2 (-), R42.2 (-), R43.2 (-), R44.2 (-), R45.2 (-), R46.2 (-), R47.2 (-), R48.2 (-); no longer D12.2 (A), D14.2 (A), D16.2 (A), D18.2 (A), D2.2 (A), D20.2 (A), D22.2 (A), D25.2 (A), D27.2 (A), D29.2 (A), D4.2 (A), D5.2 (A), D7.2 (A), D9.2 (A)
- net at Qh1.2 (B), R1.2 (-): now also R11.1 (+)
- new net: D25.2 (A), R38.1 (+)
- new net: D13.2 (A), R26.2 (-)
- new net: D23.2 (A), R31.2 (-)
- new net: D8.2 (A), R22.2 (-)
- new net: D7.2 (A), R47.1 (+)
- new net: D2.2 (A), R19.1 (+)
- new net: D16.2 (A), R42.1 (+)
- new net: D5.2 (A), R48.1 (+)
- new net: D11.2 (A), R25.2 (-)
- new net: D1.2 (A), R20.2 (-)
- new net: D21.2 (A), R30.2 (-)
- new net: D27.2 (A), R37.1 (+)
- new net: D14.2 (A), R43.1 (+)
- new net: D19.2 (A), R29.2 (-)
- new net: D18.2 (A), R41.1 (+)
- new net: D22.2 (A), R39.1 (+)
- new net: D6.2 (A), R21.2 (-)
- new net: D30.2 (A), R35.2 (-)
- new net: D26.2 (A), R33.2 (-)
- new net: D10.2 (A), R23.2 (-)
- new net: D17.2 (A), R28.2 (-)
- new net: D12.2 (A), R44.1 (+)
- new net: D9.2 (A), R46.1 (+)
- new net: D28.2 (A), R34.2 (-)
- new net: D15.2 (A), R27.2 (-)
- new net: D29.2 (A), R36.1 (+)
- new net: D4.2 (A), R45.1 (+)
- new net: D20.2 (A), R40.1 (+)
- new net bQ1A: C1.2 (-), Q2.1 (B), R10.2 (-)
- new net bQ2A: C2.2 (-), Q4.1 (B), R13.2 (-)
Other:
- moved on the sheet: D1, D10, D11, D12, D13, D14, D15, D16, D17, D18, D19, D2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

Commit message: trying to reverse engineer original circuit
Parts:
- removed Qh2: BC327, Package_TO_SOT_THT:TO-92_Inline, symbol Transistor_BJT:BC327
- removed Ql2: BC337, Package_TO_SOT_THT:TO-92_Inline, symbol Transistor_BJT:BC337
- added Qh2: MMBT2907A, Package_TO_SOT_SMD:SOT-23, symbol Transistor_BJT:MMBT3906
- added Ql2: MMBT2222A, Package_TO_SOT_SMD:SOT-23, symbol Transistor_BJT:MMBT2222A
- Qh1: value BC327 -> MMBT2907A; footprint Package_TO_SOT_THT:TO-92_Inline -> Package_TO_SOT_SMD:SOT-23; symbol Transistor_BJT:BC327 -> Transistor_BJT:MMBT3906
- Ql1: value BC337 -> MMBT2222A; footprint Package_TO_SOT_THT:TO-92_Inline -> Package_TO_SOT_SMD:SOT-23; symbol Transistor_BJT:BC337 -> Transistor_BJT:MMBT2222A
- R11, R12: value 10k -> 1k
- R14, R15: value 100 -> 1k
- R16, R17: value 10k -> 5.1k
Connections:
- net +5V: now also Qh1.2 (E), Qh2.2 (E); no longer Qh1.3 (E)
- net GND: now also Ql1.2 (E), Ql2.2 (E); no longer Ql1.3 (E)
- net H1b: now also Qh1.1 (B), R1.2 (-), R17.2 (-); no longer Q2.3 (C), Q3.3 (D), R1.1 (+), R15.1 (+), R2.1 (+), R5.2 (-)
- net H2b: now also R16.2 (-), Qh2.1 (B); no longer R12.1 (+)
- net L1b: now also Ql1.1 (B); no longer Ql1.2 (B), R16.2 (-)
- net L2b: now also Ql2.1 (B); no longer R17.2 (-)
- net LO: no longer R7.1 (+)
- net O1: now also Qh1.3 (C), Ql1.3 (C); no longer Qh1.1 (C), Ql1.1 (C)
- net O2: now also Qh2.3 (C), Ql2.3 (C)
- new net HI : Q2.3 (C), Q3.3 (D), R15.1 (+), R2.1 (+), R5.2 (-)
- now unconnected: R11.1 (+)
Other:
- moved on the sheet: R16, R17

Commit message: first appearently working prototype
Parts:
- removed Q1, Q3: AO3400A, Package_TO_SOT_SMD:SOT-23, symbol Transistor_FET:AO3400A
- removed R1, R11, R4: 1k, Resistor_SMD:R_0805_2012Metric_Pad1.20x1.40mm_HandSolder, symbol PCM_Elektuur:R
- removed R16, R17: 5.1k, Resistor_SMD:R_0805_2012Metric_Pad1.20x1.40mm_HandSolder, symbol PCM_Elektuur:R
- added C3, C4: 100p, Capacitor_SMD:C_0805_2012Metric_Pad1.18x1.45mm_HandSolder, symbol PCM_Elektuur:C
- added Q1, Q3: MMBT3904, Package_TO_SOT_SMD:SOT-23, symbol Transistor_BJT:MMBT3904
- added R18: 1k, Resistor_SMD:R_0805_2012Metric_Pad1.20x1.40mm_HandSolder, symbol PCM_Elektuur:R
- R10, R13, R6: value 1k -> 660
- R14, R15, R7: value 1k -> 330
- R5: value 100 -> 330
- R8: value 100 -> 660
- V4: value 3.3 -> 5
Connections:
- net +3.3V: no longer R6.1 (+)
- net +5V: now also R5.2 (-), R7.2 (-); no longer R12.2 (-), R5.1 (+), R8.1 (+)
- net GND: now also Q1.2 (E), Q3.2 (E)
- net H1b: now also R12.2 (-)
- net H2b: now also R18.1 (+); no longer R7.2 (-)
- net HI_IN: now also R6.1 (+), V4.1, C3.1 (+)
- net LO_IN: now also R8.1 (+), V5.1, C4.1 (+); no longer R6.2 (-)
- net at R12.1 (+): now also Q2.3 (C), R15.1 (+)
- net at R7.1 (+): now also R3.2 (-), Q3.3 (C)
- removed net HI : Q2.3 (C), R15.1 (+), R2.1 (+), R5.2 (-)
- net LO: no longer names the net of Q4.3 (C), R14.1 (+)
- net LO: now also R18.2 (-); no longer R3.2 (-), R8.2 (-)
- net bQ1A renamed bQ2
- net bQ2A renamed bQ4
- new net: Q1.3 (C), R2.1 (+), R5.1 (+)
- new net bQ1: C3.2 (-), Q1.1 (B), R6.2 (-)
- new net bQ3: C4.2 (-), Q3.1 (B), R8.2 (-)
Other:
- note added: "Dual-Transistor-Packages: MMDT2227: https://lcsc.com/product-detail/Bipolar-BJT_Diodes-Incorporated-MMDT2227-7-F_C191919.html https://lcsc.com/product-detail/Bipolar-BJT_Jiangsu-Changjing-Electronics-Technology-Co-Ltd-MMDT2227-RANGE-100-300_C35308.html ZHB6718 - komplette PNP-NPN H-Bridge bis 2.5A: https://lcsc.com/product-detail/Bipolar-BJT_Diodes-Incorporated-ZHB6718TA_C445537.html Aber: 1,56€!"
- moved on the sheet: C1, C2, D1, D10, D11, D12, D13, D14, D15, D16, D17, D18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

Commit message: change to bc807-40/817-40 and added mosfet to turn it all off
Parts:
- removed Qh2: MMBT2907A, Package_TO_SOT_SMD:SOT-23, symbol Transistor_BJT:MMBT3906
- removed Ql2: MMBT2222A, Package_TO_SOT_SMD:SOT-23, symbol Transistor_BJT:MMBT2222A
- added C5, C6: 100p, Capacitor_SMD:C_0805_2012Metric_Pad1.18x1.45mm_HandSolder, symbol PCM_Elektuur:C
- added D24, D3, D31, D32, D33, D34, D35, D36, D37, D38, D39, D40, D41, D42, D43, D44, D45, D46, D47, D48, D49, D50, D51, D52, D53, D54, D55, D56, D57, D58, D59, D60, D61, D62, D63, D64, D65, D66, D67, D68, D69, D70, D71, D72, D73, D74, D75, D76, D77, D78, D79, D80, D81, D82, D83, D84: LED, LED_THT:LED_D5.0mm, symbol Device:LED
- added Q5: AO3400A, Package_TO_SOT_SMD:SOT-23, symbol Transistor_FET:AO3400A
- added Q6: MMBT3904, Package_TO_SOT_SMD:SOT-23, symbol Transistor_BJT:MMBT3904
- added Qh2: BC807-40, Package_TO_SOT_SMD:SOT-23, symbol Transistor_BJT:BC807
- added Ql2: BC817-40, Package_TO_SOT_SMD:SOT-23, symbol Transistor_BJT:BC817
- added R1: 10, Resistor_SMD:R_0805_2012Metric_Pad1.20x1.40mm_HandSolder, symbol PCM_Elektuur:R
- added R11, R16, R17, R24, R32, R49, R50, R51, R52, R53, R54, R55, R56, R57, R58, R59, R60, R61, R62, R63, R64, R65, R66, R67, R68, R69, R70, R71, R72, R73, R74, R75, R76, R77, R78, R79, R80, R81, R82, R83, R84, R85, R86, R87, R88, R89, R90, R91, R92, R93, R94, R95, R96, R97, R98, R99: 330, Resistor_SMD:R_0805_2012Metric_Pad1.20x1.40mm_HandSolder, symbol PCM_Elektuur:R
- added R4: 1k, Resistor_SMD:R_0805_2012Metric_Pad1.20x1.40mm_HandSolder, symbol PCM_Elektuur:R
- added R9: 660, Resistor_SMD:R_0805_2012Metric_Pad1.20x1.40mm_HandSolder, symbol PCM_Elektuur:R
- added V6: VPULSE, symbol Simulation_SPICE:VPULSE
- Qh1: value MMBT2907A -> BC807-40; symbol Transistor_BJT:MMBT3906 -> Transistor_BJT:BC807
- Ql1: value MMBT2222A -> BC817-40; symbol Transistor_BJT:MMBT2222A -> Transistor_BJT:BC817
- R12, R18: value 1k -> 2k
- R14, R15, R5, R7: value 330 -> 1k
Connections:
- net +5V: now also Qh2.2 (E), R4.2 (-)
- net GND: now also Q5.2 (S), Q6.2 (E), V6.2; no longer Q1.2 (E), Q3.2 (E), Ql1.2 (E)
- net H2b: now also Qh2.1 (B)
- net L2b: now also Ql2.1 (B)
- net O1: now also D3.1 (K), D31.1 (K), D33.1 (K), D35.1 (K), D37.1 (K), D39.1 (K), D41.1 (K), D43.1 (K), D45.1 (K), D47.1 (K), D49.1 (K), D51.1 (K), D53.1 (K), D55.1 (K), D57.1 (K), D59.1 (K), D61.1 (K), D63.1 (K), D65.1 (K), D67.1 (K), D69.1 (K), D71.1 (K), D73.1 (K), D75.1 (K), D77.1 (K), D79.1 (K), D81.1 (K), D83.1 (K), R16.1 (+), R24.1 (+), R49.1 (+), R51.1 (+), R53.1 (+), R55.1 (+), R57.1 (+), R59.1 (+), R61.1 (+), R63.1 (+), R65.1 (+), R67.1 (+), R69.1 (+), R71.1 (+), R73.1 (+), R75.1 (+), R77.1 (+), R79.1 (+), R81.1 (+), R83.1 (+), R85.1 (+), R87.1 (+), R89.1 (+), R91.1 (+), R93.1 (+), R95.1 (+), R97.1 (+), R99.1 (+)
- net O2: now also D24.1 (K), D32.1 (K), D34.1 (K), D36.1 (K), D38.1 (K), D40.1 (K), D42.1 (K), D44.1 (K), D46.1 (K), D48.1 (K), D50.1 (K), D52.1 (K), D54.1 (K), D56.1 (K), D58.1 (K), D60.1 (K), D62.1 (K), D64.1 (K), D66.1 (K), D68.1 (K), D70.1 (K), D72.1 (K), D74.1 (K), D76.1 (K), D78.1 (K), D80.1 (K), D82.1 (K), D84.1 (K), Qh2.3 (C), Ql2.3 (C), R11.2 (-), R17.2 (-), R32.2 (-), R50.2 (-), R52.2 (-), R54.2 (-), R56.2 (-), R58.2 (-), R60.2 (-), R62.2 (-), R64.2 (-), R66.2 (-), R68.2 (-), R70.2 (-), R72.2 (-), R74.2 (-), R76.2 (-), R78.2 (-), R80.2 (-), R82.2 (-), R84.2 (-), R86.2 (-), R88.2 (-), R90.2 (-), R92.2 (-), R94.2 (-), R96.2 (-), R98.2 (-)
- new net: D79.2 (A), R94.1 (+)
- new net: D82.2 (A), R97.2 (-)
- new net: D59.2 (A), R74.1 (+)
- new net: D76.2 (A), R91.2 (-)
- new net: D60.2 (A), R75.2 (-)
- new net: D67.2 (A), R82.1 (+)
- new net: D68.2 (A), R83.2 (-)
- new net: D77.2 (A), R92.1 (+)
- new net: D53.2 (A), R68.1 (+)
- new net: D32.2 (A), R24.2 (-)
- new net: D41.2 (A), R56.1 (+)
- new net: D46.2 (A), R61.2 (-)
- new net: D37.2 (A), R52.1 (+)
- new net: D49.2 (A), R64.1 (+)
- new net: D84.2 (A), R99.2 (-)
- new net: D58.2 (A), R73.2 (-)
- new net: D35.2 (A), R50.1 (+)
- new net: D52.2 (A), R67.2 (-)
- new net: D3.2 (A), R11.1 (+)
- new net: D73.2 (A), R88.1 (+)
- new net: D57.2 (A), R72.1 (+)
- new net: D42.2 (A), R57.2 (-)
- new net: D36.2 (A), R51.2 (-)
- new net: D50.2 (A), R65.2 (-)
- new net: D81.2 (A), R96.1 (+)
- new net: D51.2 (A), R66.1 (+)
- new net: D47.2 (A), R62.1 (+)
- new net: D74.2 (A), R89.2 (-)
- new net: D24.2 (A), R16.2 (-)
- new net: D64.2 (A), R79.2 (-)
- new net: D54.2 (A), R69.2 (-)
- new net: D43.2 (A), R58.1 (+)
- new net: D56.2 (A), R71.2 (-)
- new net: D66.2 (A), R81.2 (-)
- new net: D61.2 (A), R76.1 (+)
- new net: D71.2 (A), R86.1 (+)
- new net: D38.2 (A), R53.2 (-)
- new net: D34.2 (A), R49.2 (-)
- new net: D48.2 (A), R63.2 (-)
- new net: D75.2 (A), R90.1 (+)
- new net: D65.2 (A), R80.1 (+)
- new net: D72.2 (A), R87.2 (-)
- new net: D62.2 (A), R77.2 (-)
- new net: D83.2 (A), R98.1 (+)
- new net: D44.2 (A), R59.2 (-)
- new net: D33.2 (A), R32.1 (+)
- new net: D55.2 (A), R70.1 (+)
- new net: D70.2 (A), R85.2 (-)
- new net: D80.2 (A), R95.2 (-)
- new net: D78.2 (A), R93.2 (-)
- new net: D69.2 (A), R84.1 (+)
- new net: D45.2 (A), R60.1 (+)
- new net: D39.2 (A), R54.1 (+)
- new net: D40.2 (A), R55.2 (-)
- new net: D31.2 (A), R17.1 (+)
- new net: D63.2 (A), R78.1 (+)
- new net EN_IN: C6.1 (+), R9.1 (+), V6.1
- new net bQ6: C6.2 (-), Q6.1 (B), R9.2 (-)
- new net drain: Q1.2 (E), Q3.2 (E), Q5.3 (D), Ql1.2 (E), Ql2.2 (E)
- new net enable: C5.1 (+), Q6.3 (C), R1.1 (+), R4.1 (+)
- new net gate: C5.2 (-), Q5.1 (G), R1.2 (-)
Other:
- moved on the sheet: C1, C2, C3, C4, D1, D10, D11, D12, D13, D14, D15, D16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

Commit message: fillet PCB and change transistor footprints
Parts:
- removed C5, C6: 100p, Capacitor_SMD:C_0805_2012Metric_Pad1.18x1.45mm_HandSolder, symbol PCM_Elektuur:C
- removed D1, D10, D11, D12, D13, D14, D15, D16, D17, D18, D19, D2, D20, D21, D22, D23, D24, D25, D26, D27, D28, D29, D3, D30, D31, D32, D33, D34, D35, D36, D37, D38, D39, D4, D40, D41, D42, D43, D44, D45, D46, D47, D48, D49, D5, D50, D51, D52, D53, D54, D55, D56, D57, D58, D59, D6, D60, D61, D62, D63, D64, D65, D66, D67, D68, D69, D7, D70, D71, D72, D73, D74, D75, D76, D77, D78, D79, D8, D80, D81, D82, D83, D84, D9: LED, LED_THT:LED_D5.0mm, symbol Device:LED
- removed Q5: AO3400A, Package_TO_SOT_SMD:SOT-23, symbol Transistor_FET:AO3400A
- removed Q6: MMBT3904, Package_TO_SOT_SMD:SOT-23, symbol Transistor_BJT:MMBT3904
- removed Qh2: BC807-40, Package_TO_SOT_SMD:SOT-23, symbol Transistor_BJT:BC807
- removed Ql2: BC817-40, Package_TO_SOT_SMD:SOT-23, symbol Transistor_BJT:BC817
- removed R1: 10, Resistor_SMD:R_0805_2012Metric_Pad1.20x1.40mm_HandSolder, symbol PCM_Elektuur:R
- removed R11, R16, R17, R19, R20, R21, R22, R23, R24, R25, R26, R27, R28, R29, R30, R31, R32, R33, R34, R35, R36, R37, R38, R39, R40, R41, R42, R43, R44, R45, R46, R47, R48, R49, R50, R51, R52, R53, R54, R55, R56, R57, R58, R59, R60, R61, R62, R63, R64, R65, R66, R67, R68, R69, R70, R71, R72, R73, R74, R75, R76, R77, R78, R79, R80, R81, R82, R83, R84, R85, R86, R87, R88, R89, R90, R91, R92, R93, R94, R95, R96, R97, R98, R99: 330, Resistor_SMD:R_0805_2012Metric_Pad1.20x1.40mm_HandSolder, symbol PCM_Elektuur:R
- removed R9: 660, Resistor_SMD:R_0805_2012Metric_Pad1.20x1.40mm_HandSolder, symbol PCM_Elektuur:R
- removed V6: VPULSE, symbol Simulation_SPICE:VPULSE
- added D1: LED_Lichterkette, LED_THT:LED_D5.0mm, symbol Device:LED_Dual_Bidirectional
- added Qh2: BC327, Package_TO_SOT_THT:TO-92_Inline, symbol Transistor_BJT:BC327
- added Ql2: BC337, Package_TO_SOT_THT:TO-92_Inline, symbol Transistor_BJT:BC337
- added R3: 220k, Resistor_SMD:R_0805_2012Metric_Pad1.20x1.40mm_HandSolder, symbol PCM_Elektuur:R
- added VMEAS1, VMEAS2: 0, symbol Simulation_SPICE:VDC
- Q1, Q2, Q3, Q4: footprint Package_TO_SOT_SMD:SOT-23 -> Package_TO_SOT_SMD:SOT-23_Handsoldering
- Qh1: value BC807-40 -> BC327; footprint Package_TO_SOT_SMD:SOT-23 -> Package_TO_SOT_THT:TO-92_Inline; symbol Transistor_BJT:BC807 -> Transistor_BJT:BC327
- Ql1: value BC817-40 -> BC337; footprint Package_TO_SOT_SMD:SOT-23 -> Package_TO_SOT_THT:TO-92_Inline; symbol Transistor_BJT:BC817 -> Transistor_BJT:BC337
- R1: renamed from R6; value 660 -> 2.2k
- R2: renamed from R10; value 660 -> 2.2k
- R4: value 1k -> 220k
- R5: renamed from R13; value 660 -> 2.2k
- R6: renamed from R8; value 660 -> 2.2k
- renumbered C3 to C1, C1 to C2, C2 to C3, R14 to R10, R5 to R11, R7 to R12, R2 to R13, R3 to R14, R15 to R7, R12 to R8, R18 to R9
Connections:
- net enable is gone; now on net GND: R4.1 (+)
- net +5V: now also Qh1.3 (E), Qh2.3 (E); no longer Qh1.2 (E), R4.2 (-)
- net GND: now also Q1.2 (E), Q3.2 (E), Ql1.3 (E), Ql2.3 (E), R3.1 (+)
- net H1b: now also Qh1.2 (B); no longer Qh1.1 (B)
- net H2b: now also Qh2.2 (B)
- net HI_IN: now also J1.4, R3.2 (-); no longer J1.3, V4.1
- net L1b: now also Ql1.2 (B); no longer Ql1.1 (B)
- net L2b: now also Ql2.2 (B)
- net LO_IN: now also J1.3, R4.2 (-), V4.1; no longer J1.4, V5.1
- net O1: now also Qh1.1 (C), Ql1.1 (C), VMEAS1.1; no longer Qh1.3 (C), Ql1.3 (C)
- net O2: now also Qh2.1 (C), Ql2.1 (C), VMEAS2.1
- removed net drain: Q1.2 (E), Q3.2 (E), Ql1.2 (E)
- new net LED_O1: D1.2 (AK), VMEAS1.2
- new net LED_O2: D1.1 (KA), VMEAS2.2
Other:
- note added: "Dual-Transistor-Packages: MMDT2227: https://lcsc.com/product-detail/Bipolar-BJT_Diodes-Incorporated-MMDT2227-7-F_C191919.html https://lcsc.com/product-detail/Bipolar-BJT_Jiangsu-Changjing-Electronics-Technology-Co-Ltd-MMDT2227-RANGE-100-300_C35308.html ZHB6718 - komplette PNP-NPN H-Bridge bis 2.5A: https://lcsc.com/product-detail/Bipolar-BJT_Diodes-Incorporated-ZHB6718TA_C445537.html Aber: 1,56€!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"
- note removed: "Dual-Transistor-Packages: MMDT2227: https://lcsc.com/product-detail/Bipolar-BJT_Diodes-Incorporated-MMDT2227-7-F_C191919.html https://lcsc.com/product-detail/Bipolar-BJT_Jiangsu-Changjing-Electronics-Technology-Co-Ltd-MMDT2227-RANGE-100-300_C35308.html ZHB6718 - komplette PNP-NPN H-Bridge bis 2.5A: https://lcsc.com/product-detail/Bipolar-BJT_Diodes-Incorporated-ZHB6718TA_C445537.html Aber: 1,56€!"
- moved on the sheet: C1, C2, C3, C4, J1, Q1, Q2, Q3, Q4, R1, R10, R11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
